Commit message: Add LIDAR

File: src/ugv/urdf/ugv.urdf.xacro (robot description, xacro)
@@ -229,4 +229,59 @@
         <axis xyz="0 1 0"/>
     </joint>
+    <!-- LiDAR sensor link -->
+    <link name="lidar_link">
+        <visual>
+        <geometry>
+            <cylinder radius="0.05" length="0.04"/>
+        </geometry>
+        <material name="black"/>
+        </visual>
+        <collision>
+        <geometry>
+            <cylinder radius="0.05" length="0.04"/>
+        </geometry>
+        </collision>
+        <inertial>
+        <mass value="0.1"/>
+        <inertia ixx="0.0001" ixy="0" ixz="0"
+                iyy="0.0001" iyz="0" izz="0.0001"/>
+        </inertial>
+    </link>
+    <!-- Mount LiDAR above the chassis -->
+    <joint name="lidar_joint" type="fixed">
+        <parent link="base_link"/>
+        <child link="lidar_link"/>
+        <origin xyz="0 0 0.14" rpy="0 0 0"/>
+    </joint>
+    <!-- Gazebo Classic ray sensor and ROS 2 LaserScan plugin -->
+    <gazebo reference="lidar_link">
+        <sensor name="ugv_lidar" type="ray">
+        <pose>0 0 0 0 0 0</pose>
+        <visualize>true</visualize>
+        <update_rate>10</update_rate>
+        <ray>
+            <scan>
+            <horizontal>
+                <samples>360</samples>
+                <resolution>1</resolution>
+                <min_angle>-3.14159</min_angle>
+                <max_angle>3.14159</max_angle>
+            </horizontal>
+            </scan>
+            <range>
+            <min>0.12</min>
+            <max>8.0</max>
+            <resolution>0.01</resolution>
+            </range>
+        </ray>
+        <plugin name="ugv_lidar_ros" filename="libgazebo_ros_ray_sensor.so">
+            <ros>
+            <remapping>~/out:=scan</remapping>
+            </ros>
+            <output_type>sensor_msgs/LaserScan</output_type>
+            <frame_name>lidar_link</frame_name>
+        </plugin>
+        </sensor>
+    </gazebo>
     <!-- ========================================================= -->
     <!-- ROS 2 Control -->

Commit message: Add UGV RL navigation and collision detection

File: src/ugv/urdf/ugv.urdf.xacro (robot description, xacro)
@@ -282,4 +282,22 @@
             <frame_name>lidar_link</frame_name>
         </plugin>
+        </sensor>
+    </gazebo>
+    <!-- Gazebo physical contact sensor -->
+    <gazebo reference="base_link">
+        <sensor name="ugv_contact_sensor" type="contact">
+            <always_on>true</always_on>
+            <update_rate>50</update_rate>
+            <visualize>false</visualize>
+            <contact>
+                <collision>base_link_collision</collision>
+            </contact>
+            <plugin name="ugv_bumper_ros" filename="libgazebo_ros_bumper.so">
+                <ros>
+                    <namespace>/ugv</namespace>
+                    <remapping>bumper_states:=contacts</remapping>
+                </ros>
+                <frame_name>base_link</frame_name>
+            </plugin>
         </sensor>
     </gazebo>

Commit message: Collision Corrected

File: src/ugv/urdf/ugv.urdf.xacro (robot description, xacro)
@@ -300,4 +300,72 @@
                 <frame_name>base_link</frame_name>
             </plugin>
+        </sensor>
+    </gazebo>
+    <!-- Contact sensor front left wheel -->
+    <gazebo reference="front_left_wheel">
+        <sensor name="front_left_contact_sensor" type="contact">
+        <always_on>true</always_on>
+        <update_rate>50</update_rate>
+        <contact>
+            <collision>front_left_wheel_collision</collision>
+        </contact>
+        <plugin name="front_left_bumper_ros" filename="libgazebo_ros_bumper.so">
+            <ros>
+            <namespace>/ugv</namespace>
+            <remapping>bumper_states:=contacts</remapping>
+            </ros>
+            <frame_name>front_left_wheel</frame_name>
+        </plugin>
+        </sensor>
+    </gazebo>
+    <!-- Contact sensor front right wheel -->
+    <gazebo reference="front_right_wheel">
+        <sensor name="front_right_contact_sensor" type="contact">
+        <always_on>true</always_on>
+        <update_rate>50</update_rate>
+        <contact>
+            <collision>front_right_wheel_collision</collision>
+        </contact>
+        <plugin name="front_right_bumper_ros" filename="libgazebo_ros_bumper.so">
+            <ros>
+            <namespace>/ugv</namespace>
+            <remapping>bumper_states:=contacts</remapping>
+            </ros>
+            <frame_name>front_right_wheel</frame_name>
+        </plugin>
+        </sensor>
+    </gazebo>
+    <!-- Contact sensor rear left wheel -->
+    <gazebo reference="rear_left_wheel">
+        <sensor name="rear_left_contact_sensor" type="contact">
+        <always_on>true</always_on>
+        <update_rate>50</update_rate>
+        <contact>
+            <collision>rear_left_wheel_collision</collision>
+        </contact>
+        <plugin name="rear_left_bumper_ros" filename="libgazebo_ros_bumper.so">
+            <ros>
+            <namespace>/ugv</namespace>
+            <remapping>bumper_states:=contacts</remapping>
+            </ros>
+            <frame_name>rear_left_wheel</frame_name>
+        </plugin>
+        </sensor>
+    </gazebo>
+    <!-- Contact sensor rear right wheel -->
+    <gazebo reference="rear_right_wheel">
+        <sensor name="rear_right_contact_sensor" type="contact">
+        <always_on>true</always_on>
+        <update_rate>50</update_rate>
+        <contact>
+            <collision>rear_right_wheel_collision</collision>
+        </contact>
+        <plugin name="rear_right_bumper_ros" filename="libgazebo_ros_bumper.so">
+            <ros>
+            <namespace>/ugv</namespace>
+            <remapping>bumper_states:=contacts</remapping>
+            </ros>
+            <frame_name>rear_right_wheel</frame_name>
+        </plugin>
         </sensor>
     </gazebo>

Commit message: Added new train and run

File: src/ugv/urdf/ugv.urdf.xacro (robot description, xacro)
@@ -2,5 +2,5 @@
 <robot name="ugv" xmlns:xacro="http://www.ros.org/wiki/xacro">
     <!-- ========================================================= -->
-    <!-- Robot dimensions -->
+    <!-- Robot dimensions (0.8m long x 0.66m wide with wheels)     -->
     <!-- ========================================================= -->
     <xacro:property name="body_length" value="0.8"/>
@@ -12,7 +12,5 @@
     <xacro:property name="wheel_y" value="0.29"/>
     <xacro:property name="wheel_z" value="-0.02"/>
-    <!-- ========================================================= -->
     <!-- Materials -->
-    <!-- ========================================================= -->
     <material name="grey">
         <color rgba="0.5 0.5 0.5 1.0"/>
@@ -22,8 +20,7 @@
     </material>
     <!-- ========================================================= -->
-    <!-- Base -->
+    <!-- Base Chassis                                              -->
     <!-- ========================================================= -->
     <link name="base_link">
-        <!-- Visual -->
         <visual>
             <origin xyz="0 0 0" rpy="0 0 0"/>
@@ -33,6 +30,5 @@
             <material name="grey"/>
         </visual>
-        <!-- Collision -->
-        <collision>
+        <collision name="base_link_collision">
             <origin xyz="0 0 0" rpy="0 0 0"/>
             <geometry>
@@ -40,213 +36,72 @@
             </geometry>
         </collision>
-        <!-- Inertia -->
         <inertial>
             <origin xyz="0 0 0" rpy="0 0 0"/>
             <mass value="10.0"/>
-            <inertia
-                ixx="0.2417"
-                ixy="0.0"
-                ixz="0.0"
-                iyy="0.5417"
-                iyz="0.0"
-                izz="0.7083"/>
+            <inertia ixx="0.2417" ixy="0.0" ixz="0.0"
+                     iyy="0.5417" iyz="0.0" izz="0.7083"/>
         </inertial>
     </link>
     <!-- ========================================================= -->
-    <!-- Front Left Wheel -->
-    <!-- ========================================================= -->
-    <link name="front_left_wheel">
-        <!-- Visual -->
+    <!-- Reusable Wheel Macro (Avoids repeating 4 identical blocks)-->
+    <!-- ========================================================= -->
+    <xacro:macro name="ugv_wheel" params="prefix x_pos y_pos">
+        <link name="${prefix}_wheel">
+            <visual>
+                <origin xyz="0 0 0" rpy="1.5708 0 0"/>
+                <geometry>
+                    <cylinder radius="${wheel_radius}" length="${wheel_width}"/>
+                </geometry>
+                <material name="black"/>
+            </visual>
+            <collision>
+                <origin xyz="0 0 0" rpy="1.5708 0 0"/>
+                <geometry>
+                    <cylinder radius="${wheel_radius}" length="${wheel_width}"/>
+                </geometry>
+            </collision>
+            <inertial>
+                <origin xyz="0 0 0" rpy="0 0 0"/>
+                <mass value="1.0"/>
+                <inertia ixx="0.00413" ixy="0.0" ixz="0.0"
+                         iyy="0.0072" iyz="0.0" izz="0.00413"/>
+            </inertial>
+        </link>
+        <joint name="${prefix}_wheel_joint" type="continuous">
+            <parent link="base_link"/>
+            <child link="${prefix}_wheel"/>
+            <origin xyz="${x_pos} ${y_pos} ${wheel_z}" rpy="0 0 0"/>
+            <axis xyz="0 1 0"/>
+        </joint>
+        <!-- Skid-steer friction high forward grip (mu1), low lateral drag (mu2) -->
+        <gazebo reference="${prefix}_wheel">
+            <mu1>1.0</mu1>
+            <mu2>0.15</mu2>
+            <kp>1000000.0</kp>
+            <kd>100.0</kd>
+            <material>Gazebo/Black</material>
+        </gazebo>
+    </xacro:macro>
+    <!-- Instantiate all 4 wheels -->
+    <xacro:ugv_wheel prefix="front_left"  x_pos="${wheel_x}"  y_pos="${wheel_y}"/>
+    <xacro:ugv_wheel prefix="front_right" x_pos="${wheel_x}"  y_pos="-${wheel_y}"/>
+    <xacro:ugv_wheel prefix="rear_left"   x_pos="-${wheel_x}" y_pos="${wheel_y}"/>
+    <xacro:ugv_wheel prefix="rear_right"  x_pos="-${wheel_x}" y_pos="-${wheel_y}"/>
+    <!-- ========================================================= -->
+    <!-- LiDAR Sensor Link (Mounted at z = 0.14m above base_link)  -->
+    <!-- ========================================================= -->
+    <link name="lidar_link">
         <visual>
-            <origin xyz="0 0 0" rpy="1.5708 0 0"/>
             <geometry>
-                <cylinder
-                    radius="${wheel_radius}"
-                    length="${wheel_width}"/>
+                <cylinder radius="0.05" length="0.04"/>
             </geometry>
             <material name="black"/>
         </visual>
-        <!-- Collision -->
-        <collision>
-            <origin xyz="0 0 0" rpy="1.5708 0 0"/>
-            <geometry>
-                <cylinder
-                    radius="${wheel_radius}"
-                    length="${wheel_width}"/>
-            </geometry>
-        </collision>
-        <!-- Inertia -->
         <inertial>
-            <origin xyz="0 0 0" rpy="0 0 0"/>
-            <mass value="1.0"/>
-            <inertia
-                ixx="0.00413"
-                ixy="0.0"
-                ixz="0.0"
-                iyy="0.0072"
-                iyz="0.0"
-                izz="0.00413"/>
+            <mass value="0.1"/>
+            <inertia ixx="0.0001" ixy="0" ixz="0"
+                     iyy="0.0001" iyz="0" izz="0.0001"/>
         </inertial>
     </link>
-    <joint name="front_left_wheel_joint" type="continuous">
-        <parent link="base_link"/>
-        <child link="front_left_wheel"/>
-        <origin
-            xyz="${wheel_x} ${wheel_y} ${wheel_z}"
-            rpy="0 0 0"/>
-        <axis xyz="0 1 0"/>
-    </joint>
-    <!-- ========================================================= -->
-    <!-- Front Right Wheel -->
-    <!-- ========================================================= -->
-    <link name="front_right_wheel">
-        <!-- Visual -->
-        <visual>
-            <origin xyz="0 0 0" rpy="1.5708 0 0"/>
-            <geometry>
-                <cylinder
-                    radius="${wheel_radius}"
-                    length="${wheel_width}"/>
-            </geometry>
-            <material name="black"/>
-        </visual>
-        <!-- Collision -->
-        <collision>
-            <origin xyz="0 0 0" rpy="1.5708 0 0"/>
-            <geometry>
-                <cylinder
-                    radius="${wheel_radius}"
-                    length="${wheel_width}"/>
-            </geometry>
-        </collision>
-        <!-- Inertia -->
-        <inertial>
-            <origin xyz="0 0 0" rpy="0 0 0"/>
-            <mass value="1.0"/>
-            <inertia
-                ixx="0.00413"
-                ixy="0.0"
-                ixz="0.0"
-                iyy="0.0072"
-                iyz="0.0"
-                izz="0.00413"/>
-        </inertial>
-    </link>
-    <joint name="front_right_wheel_joint" type="continuous">
-        <parent link="base_link"/>
-        <child link="front_right_wheel"/>
-        <origin
-            xyz="${wheel_x} -${wheel_y} ${wheel_z}"
-            rpy="0 0 0"/>
-        <axis xyz="0 1 0"/>
-    </joint>
-    <!-- ========================================================= -->
-    <!-- Rear Left Wheel -->
-    <!-- ========================================================= -->
-    <link name="rear_left_wheel">
-        <!-- Visual -->
-        <visual>
-            <origin xyz="0 0 0" rpy="1.5708 0 0"/>
-            <geometry>
-                <cylinder
-                    radius="${wheel_radius}"
-                    length="${wheel_width}"/>
-            </geometry>
-            <material name="black"/>
-        </visual>
-        <!-- Collision -->
-        <collision>
-            <origin xyz="0 0 0" rpy="1.5708 0 0"/>
-            <geometry>
-                <cylinder
-                    radius="${wheel_radius}"
-                    length="${wheel_width}"/>
-            </geometry>
-        </collision>
-        <!-- Inertia -->
-        <inertial>
-            <origin xyz="0 0 0" rpy="0 0 0"/>
-            <mass value="1.0"/>
-            <inertia
-                ixx="0.00413"
-                ixy="0.0"
-                ixz="0.0"
-                iyy="0.0072"
-                iyz="0.0"
-                izz="0.00413"/>
-        </inertial>
-    </link>
-    <joint name="rear_left_wheel_joint" type="continuous">
-        <parent link="base_link"/>
-        <child link="rear_left_wheel"/>
-        <origin
-            xyz="-${wheel_x} ${wheel_y} ${wheel_z}"
-            rpy="0 0 0"/>
-        <axis xyz="0 1 0"/>
-    </joint>
-    <!-- ========================================================= -->
-    <!-- Rear Right Wheel -->
-    <!-- ========================================================= -->
-    <link name="rear_right_wheel">
-        <!-- Visual -->
-        <visual>
-            <origin xyz="0 0 0" rpy="1.5708 0 0"/>
-            <geometry>
-                <cylinder
-                    radius="${wheel_radius}"
-                    length="${wheel_width}"/>
-            </geometry>
-            <material name="black"/>
-        </visual>
-        <!-- Collision -->
-        <collision>
-            <origin xyz="0 0 0" rpy="1.5708 0 0"/>
-            <geometry>
-                <cylinder
-                    radius="${wheel_radius}"
-                    length="${wheel_width}"/>
-            </geometry>
-        </collision>
-        <!-- Inertia -->
-        <inertial>
-            <origin xyz="0 0 0" rpy="0 0 0"/>
-            <mass value="1.0"/>
-            <inertia
-                ixx="0.00413"
-                ixy="0.0"
-                ixz="0.0"
-                iyy="0.0072"
-                iyz="0.0"
-                izz="0.00413"/>
-        </inertial>
-    </link>
-    <joint name="rear_right_wheel_joint" type="continuous">
-        <parent link="base_link"/>
-        <child link="rear_right_wheel"/>
-        <origin
-            xyz="-${wheel_x} -${wheel_y} ${wheel_z}"
-            rpy="0 0 0"/>
-        <axis xyz="0 1 0"/>
-    </joint>
-    <!-- LiDAR sensor link -->
-    <link name="lidar_link">
-        <visual>
-        <geometry>
-            <cylinder radius="0.05" length="0.04"/>
-        </geometry>
-        <material name="black"/>
-        </visual>
-        <collision>
-        <geometry>
-            <cylinder radius="0.05" length="0.04"/>
-        </geometry>
-        </collision>
-        <inertial>
-        <mass value="0.1"/>
-        <inertia ixx="0.0001" ixy="0" ixz="0"
-                iyy="0.0001" iyz="0" izz="0.0001"/>
-        </inertial>
-    </link>
-    <!-- Mount LiDAR above the chassis -->
     <joint name="lidar_joint" type="fixed">
         <parent link="base_link"/>
@@ -254,40 +109,40 @@
         <origin xyz="0 0 0.14" rpy="0 0 0"/>
     </joint>
-    <!-- Gazebo Classic ray sensor and ROS 2 LaserScan plugin -->
+    <!-- Gazebo 360 LiDAR Plugin (Updated to 30 Hz for fast RL steps) -->
     <gazebo reference="lidar_link">
         <sensor name="ugv_lidar" type="ray">
-        <pose>0 0 0 0 0 0</pose>
-        <visualize>true</visualize>
-        <update_rate>10</update_rate>
-        <ray>
-            <scan>
-            <horizontal>
-                <samples>360</samples>
-                <resolution>1</resolution>
-                <min_angle>-3.14159</min_angle>
-                <max_angle>3.14159</max_angle>
-            </horizontal>
-            </scan>
-            <range>
-            <min>0.12</min>
-            <max>8.0</max>
-            <resolution>0.01</resolution>
-            </range>
-        </ray>
-        <plugin name="ugv_lidar_ros" filename="libgazebo_ros_ray_sensor.so">
-            <ros>
-            <remapping>~/out:=scan</remapping>
-            </ros>
-            <output_type>sensor_msgs/LaserScan</output_type>
-            <frame_name>lidar_link</frame_name>
-        </plugin>
+            <pose>0 0 0 0 0 0</pose>
+            <visualize>true</visualize>
+            <update_rate>30</update_rate>
+            <ray>
+                <scan>
+                    <horizontal>
+                        <samples>360</samples>
+                        <resolution>1</resolution>
+                        <min_angle>-3.14159</min_angle>
+                        <max_angle>3.14159</max_angle>
+                    </horizontal>
+                </scan>
+                <range>
+                    <min>0.12</min>
+                    <max>8.0</max>
+                    <resolution>0.01</resolution>
+                </range>
+            </ray>
+            <plugin name="ugv_lidar_ros" filename="libgazebo_ros_ray_sensor.so">
+                <ros>
+                    <remapping>~/out:=scan</remapping>
+                </ros>
+                <output_type>sensor_msgs/LaserScan</output_type>
+                <frame_name>lidar_link</frame_name>
+            </plugin>
         </sensor>
     </gazebo>
-    <!-- Gazebo physical contact sensor -->
+    <!-- Single Chassis Contact Sensor (No wheel ground-contact spam) -->
     <gazebo reference="base_link">
+        <material>Gazebo/Grey</material>
         <sensor name="ugv_contact_sensor" type="contact">
             <always_on>true</always_on>
             <update_rate>50</update_rate>
-            <visualize>false</visualize>
             <contact>
                 <collision>base_link_collision</collision>
@@ -302,74 +157,6 @@
         </sensor>
     </gazebo>
-    <!-- Contact sensor front left wheel -->
-    <gazebo reference="front_left_wheel">
-        <sensor name="front_left_contact_sensor" type="contact">
-        <always_on>true</always_on>
-        <update_rate>50</update_rate>
-        <contact>
-            <collision>front_left_wheel_collision</collision>
-        </contact>
-        <plugin name="front_left_bumper_ros" filename="libgazebo_ros_bumper.so">
-            <ros>
-            <namespace>/ugv</namespace>
-            <remapping>bumper_states:=contacts</remapping>
-            </ros>
-            <frame_name>front_left_wheel</frame_name>
-        </plugin>
-        </sensor>
-    </gazebo>
-    <!-- Contact sensor front right wheel -->
-    <gazebo reference="front_right_wheel">
-        <sensor name="front_right_contact_sensor" type="contact">
-        <always_on>true</always_on>
-        <update_rate>50</update_rate>
-        <contact>
-            <collision>front_right_wheel_collision</collision>
-        </contact>
-        <plugin name="front_right_bumper_ros" filename="libgazebo_ros_bumper.so">
-            <ros>
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